Commit message: [xsturret_descriptions] Update model mesh files, add gazebo, control xacros

File: interbotix_ros_xsturrets/interbotix_xsturret_descriptions/urdf/pxxls.urdf.xacro (robot description, xacro)
@@ -23,7 +23,4 @@
     <texture filename="package://interbotix_xsturret_descriptions/meshes/interbotix_black.png"/>
   </material>
-  <xacro:if value="${hardware_type == 'gz_classic'}">
-    <xacro:include filename="$(find interbotix_xsturret_gazebo)/config/interbotix_texture.gazebo"/>
-  </xacro:if>  <!-- hardware_type == 'gz_classic' -->
   <xacro:if value="$(arg use_world_frame)">
     <link name="world"/>
@@ -42,5 +39,5 @@
       <geometry>
         <mesh
-          filename="${mesh_directory}/pxxls_base.stl"
+          filename="${mesh_directory}/base.stl"
           scale="0.001 0.001 0.001"/>
       </geometry>
@@ -53,5 +50,5 @@
       <geometry>
         <mesh
-          filename="${mesh_directory}/pxxls_base.stl"
+          filename="${mesh_directory}/base.stl"
           scale="0.001 0.001 0.001"/>
       </geometry>
@@ -93,5 +90,5 @@
       <geometry>
         <mesh
-          filename="${mesh_directory}/pxxls_pan.stl"
+          filename="${mesh_directory}/pan.stl"
           scale="0.001 0.001 0.001"/>
       </geometry>
@@ -104,5 +101,5 @@
       <geometry>
         <mesh
-          filename="${mesh_directory}/pxxls_pan.stl"
+          filename="${mesh_directory}/pan.stl"
           scale="0.001 0.001 0.001"/>
       </geometry>
@@ -144,5 +141,5 @@
       <geometry>
         <mesh
-          filename="${mesh_directory}/pxxls_tilt.stl"
+          filename="${mesh_directory}/tilt.stl"
           scale="0.001 0.001 0.001"/>
       </geometry>
@@ -155,5 +152,5 @@
       <geometry>
         <mesh
-          filename="${mesh_directory}/pxxls_tilt.stl"
+          filename="${mesh_directory}/tilt.stl"
           scale="0.001 0.001 0.001"/>
       </geometry>
@@ -185,4 +182,9 @@
   <link name="$(arg robot_name)/surface_link">
   </link>
+  <xacro:include filename="$(find interbotix_xsturret_descriptions)/urdf/control.urdf.xacro"/>
+  <xacro:include filename="$(find interbotix_xsturret_descriptions)/urdf/gazebo_configs.urdf.xacro"/>
+  <xacro:if value="${hardware_type == 'gz_classic'}">
+    <xacro:gazebo_configs/>
+  </xacro:if>
   <xacro:if value="${urdf_loc != ''}">
     <xacro:include filename="${urdf_loc}"/>

File: interbotix_ros_xsturrets/interbotix_xsturret_descriptions/urdf/pxxls_cam.urdf.xacro (robot description, xacro)
@@ -8,7 +8,8 @@
   <xacro:arg name="use_world_frame"           default="false"/>
   <xacro:arg name="external_urdf_loc"         default=""/>
-  <xacro:arg name="load_gazebo_configs"       default="false"/>
+  <xacro:arg name="hardware_type"             default="actual"/>
   <xacro:property name="mesh_directory"       value="package://interbotix_xsturret_descriptions/meshes/${robot_model}_meshes"/>
   <xacro:property name="urdf_loc"             value="$(arg external_urdf_loc)"/>
+  <xacro:property name="hardware_type"        value="$(arg hardware_type)"/>
   <xacro:property name="pan_limit_effort"     value="3"/>
   <xacro:property name="pan_limit_lower"      value="-3.14"/>
@@ -22,7 +23,4 @@
     <texture filename="package://interbotix_xsturret_descriptions/meshes/interbotix_black.png"/>
   </material>
-  <xacro:if value="$(arg load_gazebo_configs)">
-    <xacro:include filename="$(find interbotix_xsturret_gazebo)/config/interbotix_texture.gazebo"/>
-  </xacro:if>
   <xacro:if value="$(arg use_world_frame)">
     <link name="world"/>
@@ -41,16 +39,16 @@
       <geometry>
         <mesh
-          filename="${mesh_directory}/pxxls_cam_base.stl"
-          scale="0.001 0.001 0.001"/>
-      </geometry>
-      <material name="interbotix_black"/>
-    </visual>
-    <collision>
-      <origin
-        rpy="0 0 ${pi/2}"
-        xyz="0 0 0"/>
-      <geometry>
-        <mesh
-          filename="${mesh_directory}/pxxls_cam_base.stl"
+          filename="${mesh_directory}/base.stl"
+          scale="0.001 0.001 0.001"/>
+      </geometry>
+      <material name="interbotix_black"/>
+    </visual>
+    <collision>
+      <origin
+        rpy="0 0 ${pi/2}"
+        xyz="0 0 0"/>
+      <geometry>
+        <mesh
+          filename="${mesh_directory}/base.stl"
           scale="0.001 0.001 0.001"/>
       </geometry>
@@ -92,5 +90,5 @@
       <geometry>
         <mesh
-          filename="${mesh_directory}/pxxls_cam_pan.stl"
+          filename="${mesh_directory}/pan.stl"
           scale="0.001 0.001 0.001"/>
       </geometry>
@@ -103,5 +101,5 @@
       <geometry>
         <mesh
-          filename="${mesh_directory}/pxxls_cam_pan.stl"
+          filename="${mesh_directory}/pan.stl"
           scale="0.001 0.001 0.001"/>
       </geometry>
@@ -143,16 +141,16 @@
       <geometry>
         <mesh
-          filename="${mesh_directory}/pxxls_cam_tilt.stl"
-          scale="0.001 0.001 0.001"/>
-      </geometry>
-      <material name="interbotix_black"/>
-    </visual>
-    <collision>
-      <origin
-        rpy="0 0 0"
-        xyz="0 0 0"/>
-      <geometry>
-        <mesh
-          filename="${mesh_directory}/pxxls_cam_tilt.stl"
+          filename="${mesh_directory}/tilt.stl"
+          scale="0.001 0.001 0.001"/>
+      </geometry>
+      <material name="interbotix_black"/>
+    </visual>
+    <collision>
+      <origin
+        rpy="0 0 0"
+        xyz="0 0 0"/>
+      <geometry>
+        <mesh
+          filename="${mesh_directory}/tilt.stl"
           scale="0.001 0.001 0.001"/>
       </geometry>
@@ -200,20 +198,25 @@
       <geometry>
         <mesh
-          filename="${mesh_directory}/pxxls_cam_camera.stl"
-          scale="0.001 0.001 0.001"/>
-      </geometry>
-      <material name="interbotix_black"/>
-    </visual>
-    <collision>
-      <origin
-        rpy="0 0 0"
-        xyz="0 0 0"/>
-      <geometry>
-        <mesh
-          filename="${mesh_directory}/pxxls_cam_camera.stl"
-          scale="0.001 0.001 0.001"/>
-      </geometry>
-    </collision>
-  </link>
+          filename="${mesh_directory}/camera.stl"
+          scale="0.001 0.001 0.001"/>
+      </geometry>
+      <material name="interbotix_black"/>
+    </visual>
+    <collision>
+      <origin
+        rpy="0 0 0"
+        xyz="0 0 0"/>
+      <geometry>
+        <mesh
+          filename="${mesh_directory}/camera.stl"
+          scale="0.001 0.001 0.001"/>
+      </geometry>
+    </collision>
+  </link>
+  <xacro:include filename="$(find interbotix_xsturret_descriptions)/urdf/control.urdf.xacro"/>
+  <xacro:include filename="$(find interbotix_xsturret_descriptions)/urdf/gazebo_configs.urdf.xacro"/>
+  <xacro:if value="${hardware_type == 'gz_classic'}">
+    <xacro:gazebo_configs/>
+  </xacro:if>
   <xacro:if value="${urdf_loc != ''}">
     <xacro:include filename="${urdf_loc}"/>

File: interbotix_ros_xsturrets/interbotix_xsturret_descriptions/urdf/vxxmd.urdf.xacro (robot description, xacro)
@@ -23,7 +23,4 @@
     <texture filename="package://interbotix_xsturret_descriptions/meshes/interbotix_black.png"/>
   </material>
-  <xacro:if value="${hardware_type == 'gz_classic'}">
-    <xacro:include filename="$(find interbotix_xsturret_gazebo)/config/interbotix_texture.gazebo"/>
-  </xacro:if>  <!-- hardware_type == 'gz_classic' -->
   <xacro:if value="$(arg use_world_frame)">
     <link name="world"/>
@@ -42,5 +39,5 @@
       <geometry>
         <mesh
-          filename="${mesh_directory}/vxxmd_base.stl"
+          filename="${mesh_directory}/base.stl"
           scale="0.001 0.001 0.001"/>
       </geometry>
@@ -53,5 +50,5 @@
       <geometry>
         <mesh
-          filename="${mesh_directory}/vxxmd_base.stl"
+          filename="${mesh_directory}/base.stl"
           scale="0.001 0.001 0.001"/>
       </geometry>
@@ -93,5 +90,5 @@
       <geometry>
         <mesh
-          filename="${mesh_directory}/vxxmd_pan.stl"
+          filename="${mesh_directory}/pan.stl"
           scale="0.001 0.001 0.001"/>
       </geometry>
@@ -104,5 +101,5 @@
       <geometry>
         <mesh
-          filename="${mesh_directory}/vxxmd_pan.stl"
+          filename="${mesh_directory}/pan.stl"
           scale="0.001 0.001 0.001"/>
       </geometry>
@@ -144,5 +141,5 @@
       <geometry>
         <mesh
-          filename="${mesh_directory}/vxxmd_tilt.stl"
+          filename="${mesh_directory}/tilt.stl"
           scale="0.001 0.001 0.001"/>
       </geometry>
@@ -155,5 +152,5 @@
       <geometry>
         <mesh
-          filename="${mesh_directory}/vxxmd_tilt.stl"
+          filename="${mesh_directory}/tilt.stl"
           scale="0.001 0.001 0.001"/>
       </geometry>
@@ -185,4 +182,9 @@
   <link name="$(arg robot_name)/surface_link">
   </link>
+  <xacro:include filename="$(find interbotix_xsturret_descriptions)/urdf/control.urdf.xacro"/>
+  <xacro:include filename="$(find interbotix_xsturret_descriptions)/urdf/gazebo_configs.urdf.xacro"/>
+  <xacro:if value="${hardware_type == 'gz_classic'}">
+    <xacro:gazebo_configs/>
+  </xacro:if>
   <xacro:if value="${urdf_loc != ''}">
     <xacro:include filename="${urdf_loc}"/>

File: interbotix_ros_xsturrets/interbotix_xsturret_descriptions/urdf/vxxms.urdf.xacro (robot description, xacro)
@@ -23,7 +23,4 @@
     <texture filename="package://interbotix_xsturret_descriptions/meshes/interbotix_black.png"/>
   </material>
-  <xacro:if value="${hardware_type == 'gz_classic'}">
-    <xacro:include filename="$(find interbotix_xsturret_gazebo)/config/interbotix_texture.gazebo"/>
-  </xacro:if>  <!-- hardware_type == 'gz_classic' -->
   <xacro:if value="$(arg use_world_frame)">
     <link name="world"/>
@@ -42,5 +39,5 @@
       <geometry>
         <mesh
-          filename="${mesh_directory}/vxxms_base.stl"
+          filename="${mesh_directory}/base.stl"
           scale="0.001 0.001 0.001"/>
       </geometry>
@@ -53,5 +50,5 @@
       <geometry>
         <mesh
-          filename="${mesh_directory}/vxxms_base.stl"
+          filename="${mesh_directory}/base.stl"
           scale="0.001 0.001 0.001"/>
       </geometry>
@@ -93,5 +90,5 @@
       <geometry>
         <mesh
-          filename="${mesh_directory}/vxxms_pan.stl"
+          filename="${mesh_directory}/pan.stl"
           scale="0.001 0.001 0.001"/>
       </geometry>
@@ -104,5 +101,5 @@
       <geometry>
         <mesh
-          filename="${mesh_directory}/vxxms_pan.stl"
+          filename="${mesh_directory}/pan.stl"
           scale="0.001 0.001 0.001"/>
       </geometry>
@@ -144,5 +141,5 @@
       <geometry>
         <mesh
-          filename="${mesh_directory}/vxxms_tilt.stl"
+          filename="${mesh_directory}/tilt.stl"
           scale="0.001 0.001 0.001"/>
       </geometry>
@@ -155,5 +152,5 @@
       <geometry>
         <mesh
-          filename="${mesh_directory}/vxxms_tilt.stl"
+          filename="${mesh_directory}/tilt.stl"
           scale="0.001 0.001 0.001"/>
       </geometry>
@@ -185,4 +182,9 @@
   <link name="$(arg robot_name)/surface_link">
   </link>
+  <xacro:include filename="$(find interbotix_xsturret_descriptions)/urdf/control.urdf.xacro"/>
+  <xacro:include filename="$(find interbotix_xsturret_descriptions)/urdf/gazebo_configs.urdf.xacro"/>
+  <xacro:if value="${hardware_type == 'gz_classic'}">
+    <xacro:gazebo_configs/>
+  </xacro:if>
   <xacro:if value="${urdf_loc != ''}">
     <xacro:include filename="${urdf_loc}"/>

File: interbotix_ros_xsturrets/interbotix_xsturret_descriptions/urdf/wxxmd.urdf.xacro (robot description, xacro)
@@ -23,7 +23,4 @@
     <texture filename="package://interbotix_xsturret_descriptions/meshes/interbotix_black.png"/>
   </material>
-  <xacro:if value="${hardware_type == 'gz_classic'}">
-    <xacro:include filename="$(find interbotix_xsturret_gazebo)/config/interbotix_texture.gazebo"/>
-  </xacro:if>  <!-- hardware_type == 'gz_classic' -->
   <xacro:if value="$(arg use_world_frame)">
     <link name="world"/>
@@ -42,5 +39,5 @@
       <geometry>
         <mesh
-          filename="${mesh_directory}/wxxmd_base.stl"
+          filename="${mesh_directory}/base.stl"
           scale="0.001 0.001 0.001"/>
       </geometry>
@@ -53,5 +50,5 @@
       <geometry>
         <mesh
-          filename="${mesh_directory}/wxxmd_base.stl"
+          filename="${mesh_directory}/base.stl"
           scale="0.001 0.001 0.001"/>
       </geometry>
@@ -93,5 +90,5 @@
       <geometry>
         <mesh
-          filename="${mesh_directory}/wxxmd_pan.stl"
+          filename="${mesh_directory}/pan.stl"
           scale="0.001 0.001 0.001"/>
       </geometry>
@@ -104,5 +101,5 @@
       <geometry>
         <mesh
-          filename="${mesh_directory}/wxxmd_pan.stl"
+          filename="${mesh_directory}/pan.stl"
           scale="0.001 0.001 0.001"/>
       </geometry>
@@ -144,5 +141,5 @@
       <geometry>
         <mesh
-          filename="${mesh_directory}/wxxmd_tilt.stl"
+          filename="${mesh_directory}/tilt.stl"
           scale="0.001 0.001 0.001"/>
       </geometry>
@@ -155,5 +152,5 @@
       <geometry>
         <mesh
-          filename="${mesh_directory}/wxxmd_tilt.stl"
+          filename="${mesh_directory}/tilt.stl"
           scale="0.001 0.001 0.001"/>
       </geometry>
@@ -185,4 +182,9 @@
   <link name="$(arg robot_name)/surface_link">
   </link>
+  <xacro:include filename="$(find interbotix_xsturret_descriptions)/urdf/control.urdf.xacro"/>
+  <xacro:include filename="$(find interbotix_xsturret_descriptions)/urdf/gazebo_configs.urdf.xacro"/>
+  <xacro:if value="${hardware_type == 'gz_classic'}">
+    <xacro:gazebo_configs/>
+  </xacro:if>
   <xacro:if value="${urdf_loc != ''}">
     <xacro:include filename="${urdf_loc}"/>

File: interbotix_ros_xsturrets/interbotix_xsturret_descriptions/urdf/wxxms.urdf.xacro (robot description, xacro)
@@ -23,7 +23,4 @@
     <texture filename="package://interbotix_xsturret_descriptions/meshes/interbotix_black.png"/>
   </material>
-  <xacro:if value="${hardware_type == 'gz_classic'}">
-    <xacro:include filename="$(find interbotix_xsturret_gazebo)/config/interbotix_texture.gazebo"/>
-  </xacro:if>  <!-- hardware_type == 'gz_classic' -->
   <xacro:if value="$(arg use_world_frame)">
     <link name="world"/>
@@ -42,5 +39,5 @@
       <geometry>
         <mesh
-          filename="${mesh_directory}/wxxms_base.stl"
+          filename="${mesh_directory}/base.stl"
           scale="0.001 0.001 0.001"/>
       </geometry>
@@ -53,5 +50,5 @@
       <geometry>
         <mesh
-          filename="${mesh_directory}/wxxms_base.stl"
+          filename="${mesh_directory}/base.stl"
           scale="0.001 0.001 0.001"/>
       </geometry>
@@ -93,5 +90,5 @@
       <geometry>
         <mesh
-          filename="${mesh_directory}/wxxms_pan.stl"
+          filename="${mesh_directory}/pan.stl"
           scale="0.001 0.001 0.001"/>
       </geometry>
@@ -104,5 +101,5 @@
       <geometry>
         <mesh
-          filename="${mesh_directory}/wxxms_pan.stl"
+          filename="${mesh_directory}/pan.stl"
           scale="0.001 0.001 0.001"/>
       </geometry>
@@ -144,5 +141,5 @@
       <geometry>
         <mesh
-          filename="${mesh_directory}/wxxms_tilt.stl"
+          filename="${mesh_directory}/tilt.stl"
           scale="0.001 0.001 0.001"/>
       </geometry>
@@ -155,5 +152,5 @@
       <geometry>
         <mesh
-          filename="${mesh_directory}/wxxms_tilt.stl"
+          filename="${mesh_directory}/tilt.stl"
           scale="0.001 0.001 0.001"/>
       </geometry>
@@ -185,4 +182,9 @@
   <link name="$(arg robot_name)/surface_link">
   </link>
+  <xacro:include filename="$(find interbotix_xsturret_descriptions)/urdf/control.urdf.xacro"/>
+  <xacro:include filename="$(find interbotix_xsturret_descriptions)/urdf/gazebo_configs.urdf.xacro"/>
+  <xacro:if value="${hardware_type == 'gz_classic'}">
+    <xacro:gazebo_configs/>
+  </xacro:if>
   <xacro:if value="${urdf_loc != ''}">
     <xacro:include filename="${urdf_loc}"/>
